File: boardwright.kicad_pcb (KiCad board)
At the start: 6 copper layers, 0 parts

Commit message: feat(hardware): add Boardwright CI fixture circuit
Parts:
- added D1: LED, LED_THT:LED_D5.0mm_FlatTop, F.Cu at (151.0, 80.0)
- added R1: R, Resistor_THT:R_Axial_DIN0617_L17.0mm_D6.0mm_P30.48mm_Horizontal, F.Cu at (159.2, 88.8)
- added TP1: TestPoint, RD-Testpoints:TestPoint_Pad_D1.5mm, F.Cu at (145.0, 72.0)
- added U1: NE555D, Package_SO:SOIC-8_3.9x4.9mm_P1.27mm, F.Cu at (158.0, 69.0)
Other:
- board outline added: 59 x 32 mm
- board text removed: "30°"
- board text removed: "3× 120°"
